File: Project/Test/Test.kicad_sch (KiCad schematic)
At the start: 159 parts, among them J1 DC Power Jack 2.1mm - PCB Mou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, J10 TO5 Transistor Socket - 3 Pin, J2 1x4 Header 2.54mm, J3 NMJ4HCD2, J4 NMJ6HCD2, J5 DIP8 IC Socket - 8 Pin, J6 DIP14 IC Socket - 14 Pin, J7 DIP16 IC Socket - 16 Pin, J8 Pin Header Socket - 20 pin, J9 SIP36 - 36 Pin Snappable In-l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, Q1 2N5088, Q10 2N5089, Q11 BC108C, Q12 BC108, Q13 2SC1815GR, Q14 BC549B, Q15 MPSA18, Q16 2N7000, Q17 2N5458, Q18 BC183B, Q19 BC109, Q2 2N5087, Q20 BC108B, Q21 BC108, Q22 BC109C, Q23 BC549C, Q24 2N2222A, Q25 2N5457, Q26 MPS751, Q27 MPS8599, Q28 J113, Q29 J201, Q3 MPSA13, Q30 J202, Q31 2N1613, Q32 PF5102, Q33 GT402, Q34 MP42B, Q35 MMBFJ201, Q36 MMBF5457, Q4 BC550B, Q5 BS170, Q6 2N3904, Q7 2N3906, Q8 2N4125, Q9 2N4401, SW1 DIP Switch - 2 Position, SW10 DPDT Toggle Switch ON/ON - PC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, SW11 DPDT Toggle Switch ON/ON/ON -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, SW12 DPDT Sub Mini Toggle Switch -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, SW13 DPDT Sub Mini Toggle Switch -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, SW14 DPDT Sub Mini Toggle Switch -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, SW2 DIP Switch - 3 Position, SW3 DIP Switch - 4 Position, SW4 DIP Switch - 6 Position, SW5 DIP Switch - 12 Position, SW6 3PDT Footswitch - PCB Pin - A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, SW7 3PDT Footswitch PRO - PCB Pin, SW8 SPDT Toggle Switch ON/ON - PC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, SW9 SPDT Toggle Switch ON/OFF/ON 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, T1 TY-141P, T2 42TM018-RC, U1 CD4044BE, U10 MC1496P, U11 CD4069UBE, U12 TL062CP, U13 LM833N, U14 CD4007CN, U15 TL072IP, U16 NE555P, U17 CAT24C32LI-G, U18 LM380N, U19 JRC4558D, U2 V2153M, U20 CA3080AE, U21 PT2399, U22 LM386N-3, U23 OPA2134PA, U24 TL071, U25 LT1054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

Commit message: Update
Parts:
- removed R2: 1/4W Metal Film Resistor, Library:R_10.16mm_H, symbol Library:RES-QW
- removed R3: 1/4W Metal Film Resistor, Library:R_10.16mm_H, symbol Library:RES-QW-BAG
- added B1: 125B, Library:125B, symbol Library:Case_125B
- added B2: 1590B, Library:1590B, symbol Library:Case_1590B
- added B3: 1590BB, Library:1590BB, symbol Library:Case_1590BB
- added R2: 1/4W P7.62, Library:R_7.62mm_H, symbol Library:RES_7.62
- added R3: 1/4W P10.16, Library:R_10.16mm_H, symbol Library:RES_10.16
Other:
- note added: "Caps"
- note added: "Cases"
- note added: "Diodes"
- note added: "Dip Switches"
- note added: "Headers"
- note added: "IC"
- note added: "IC Sockets"
- note added: "Jacks"
- note added: "Pots"
- note added: "RES"
- note added: "Switches"
- note added: "Testpads"
- note added: "Transformers and Inductors"
- note added: "Transistors"
- moved on the sheet: 1, C1, C10, C11, C12, C13, C14, C2, C3, C4, C5, C6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
